File: box_plate/box_plate.kicad_pcb (KiCad board)
At the start: 2 copper layers, 149.9 x 146.8 mm, 9 parts, among them J1 Conn_02x04_Odd_Even, U1 PWR_ACDC, U2 RELAY_4CH, U3 RSL10_EVK

Commit message: Updated PCB files.
Parts:
- removed R1: 0, Resistor_THT:R_Axial_DIN0204_L3.6mm_D1.6mm_P7.62mm_Horizontal
- added J2: Conn_02x04_Odd_Even, Connector_PinHeader_2.54mm:PinHeader_2x04_P2.54mm_Vertical, F.Cu at (181.6, 195.6)
- moved J1 41.5 mm to (270.5, 176.5), turned to 180 degrees
Connections:
- J1 pad 1: Net-(J1-Pad1) -> +3V3
- J1 pad 2: Net-(J1-Pad1) -> +3V3
- J1 pad 3: Net-(J1-Pad3) -> /DIO4
- J1 pad 4: Net-(J1-Pad4) -> /DIO14
- J1 pad 5: Net-(J1-Pad5) -> /DIO5
- J1 pad 6: Net-(J1-Pad6) -> /DIO13
- U2 pad 2: Net-(U2-Pad2) -> /DIO0
- U2 pad 3: Net-(U2-Pad3) -> /DIO1
- U2 pad 4: Net-(U2-Pad4) -> /DIO2
- U2 pad 5: Net-(U2-Pad5) -> /DIO3
- U3 pad 10: Net-(U2-Pad2) -> /DIO1
- U3 pad 11: Net-(U3-Pad11) -> /DIO2
- U3 pad 12: Net-(U3-Pad12) -> /DIO3
- U3 pad 15: Net-(J1-Pad4) -> /DIO4
- U3 pad 16: Net-(J1-Pad6) -> /DIO5
- U3 pad 19: Net-(J1-Pad3) -> /DIO13
- U3 pad 20: Net-(J1-Pad5) -> /DIO14
- U3 pad 9: Net-(U2-Pad5) -> /DIO0
Routing:
- net GND: track 214.2 -> 501.2 mm
- net GNDA: track 0.00 -> 136.9 mm
- net +12V: track 0.00 -> 123.8 mm
- net /DIO14: track 0.00 -> 95.7 mm
- net /DIO13: track 0.00 -> 93.6 mm
- net /DIO4: track 0.00 -> 88.9 mm
- net /DIO5: track 0.00 -> 87.1 mm
- net Net-(J1-Pad5): track 69.4 -> 0.00 mm
- net Net-(J1-Pad3): track 67.9 -> 0.00 mm
- net +3V3: track 20.6 -> 82.0 mm
- net Net-(U2-Pad2): track 51.8 -> 0.00 mm
- net Net-(J1-Pad6): track 49.9 -> 0.00 mm
- net /DIO3: track 0.00 -> 45.7 mm
- net /DIO2: track 0.00 -> 45.4 mm
- net /DIO0: track 0.00 -> 45.4 mm
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Other:
- net class Default: clearance 0.508 -> 0.381; trace_width 0.4064 -> 0.381
- net class Power added: clearance 0.762, trace_width 0.762, via_dia 0.8, via_drill 0.4
- rule trace_clearance: 0.508 -> 0.381
